Commit message: intergrate yolo, nav2, slam, pipeline

File: lidar_robot/urdf/robot.urdf.xacro (robot description, xacro)
@@ -118,3 +118,20 @@
     <origin xyz="0.1 0.0 ${body_height/2 + 0.025}" rpy="0 0 0"/>
   </joint>
+  <!-- Camera Joint -->
+  <joint name="camera_joint" type="fixed">
+    <parent link="base_link"/>
+    <child link="camera_link"/>
+    <origin xyz="0.15 0 0.1" rpy="0 0 0"/>
+  </joint>
+  <!-- Camera Link -->
+  <link name="camera_link">
+    <visual>
+      <geometry>
+        <box size="0.05 0.05 0.05"/>
+      </geometry>
+      <material name="red">
+        <color rgba="1.0 0.0 0.0 1.0"/>
+      </material>
+    </visual>
+  </link>
 </robot>
